Commit message: Fixed Gazebo with updated version (Gazebo Harmonic) (Dude this took me HOURS this is insane)

File: description/robot_core.xacro (robot description, xacro)
@@ -66,12 +66,5 @@
         </xacro:inertial_box>
     </link>
-    <gazebo reference="chassis">
-        <material>
-            <script>
-                <uri>file://media/materials/scripts/gazebo.material</uri>
-                <name>Gazebo/Blue</name>
-            </script>
-        </material>
-    </gazebo>
+    <gazebo reference="chassis"/>
     <!-- LEFT WHEEL LINK -->
     <joint name="left_wheel_joint" type="continuous">
@@ -97,12 +90,5 @@
         </xacro:inertial_cylinder>
     </link>
-    <gazebo reference="left_wheel">
-        <!-- <material>
-            <script>
-                <uri>file://media/materials/scripts/gazebo.material</uri>
-                <name>Gazebo/Blue</name>
-            </script>
-        </material> -->
-    </gazebo>
+    <gazebo reference="left_wheel"/>
     <!-- RIGHT WHEEL LINK -->
     <joint name="right_wheel_joint" type="continuous">
@@ -128,12 +114,5 @@
         </xacro:inertial_cylinder>
     </link>
-    <gazebo reference="right_wheel">
-        <!-- <material>
-            <script>
-                <uri>file://media/materials/scripts/gazebo.material</uri>
-                <name>Gazebo/Blue</name>
-            </script>
-        </material> -->
-    </gazebo>
+    <gazebo reference="right_wheel"/>
     <!-- CASTER WHEEL LINK -->
     <joint name="caster_wheel_joint" type="fixed">
@@ -159,10 +138,4 @@
     </link>
     <gazebo reference="caster_wheel">
-        <!-- <material>
-            <script>
-                <uri>file://media/materials/scripts/gazebo.material</uri>
-                <name>Gazebo/White</name>
-            </script>
-        </material> -->
         <mu1 value="0.001"/>
         <mu2 value="0.001"/>
